Commit message: changes to urdf added radar link

File: husky_description/urdf/husky.urdf.xacro (robot description, xacro)
@@ -26,4 +26,58 @@
         <update_rate>100</update_rate>
         <visualize>true</visualize>
+        <!-- <imu>
+          <angular_velocity>
+            <x>
+              <noise type="gaussian">
+                <mean>0.0</mean>
+                <stddev>2e-4</stddev>
+                <bias_mean>0.0000075</bias_mean>
+                <bias_stddev>0.0000008</bias_stddev>
+              </noise>
+            </x>
+            <y>
+              <noise type="gaussian">
+                <mean>0.0</mean>
+                <stddev>2e-4</stddev>
+                <bias_mean>0.0000075</bias_mean>
+                <bias_stddev>0.0000008</bias_stddev>
+              </noise>
+            </y>
+            <z>
+              <noise type="gaussian">
+                <mean>0.0</mean>
+                <stddev>2e-4</stddev>
+                <bias_mean>0.0000075</bias_mean>
+                <bias_stddev>0.0000008</bias_stddev>
+              </noise>
+            </z>
+          </angular_velocity>
+          <linear_acceleration>
+            <x>
+              <noise type="gaussian">
+                <mean>0.0</mean>
+                <stddev>1.7e-2</stddev>
+                <bias_mean>0.1</bias_mean>
+                <bias_stddev>0.001</bias_stddev>
+              </noise>
+            </x>
+            <y>
+              <noise type="gaussian">
+                <mean>0.0</mean>
+                <stddev>1.7e-2</stddev>
+                <bias_mean>0.1</bias_mean>
+                <bias_stddev>0.001</bias_stddev>
+              </noise>
+            </y>
+            <z>
+              <noise type="gaussian">
+                <mean>0.0</mean>
+                <stddev>1.7e-2</stddev>
+                <bias_mean>0.1</bias_mean>
+                <bias_stddev>0.001</bias_stddev>
+              </noise>
+            </z>
+          </linear_acceleration>
+        </imu>         -->
       </sensor>
     </gazebo>

File: husky_description/urdf/husky_macro.urdf.xacro (robot description, xacro)
@@ -89,4 +89,26 @@
       <child link="${prefix}gps_link" />
     </joint>
+  <link name="/radar_link">
+        <visual>
+            <origin xyz="0 0 0" rpy="0 0 0"/>
+            <geometry>
+                <box size="0.05 0.1 0.1"/>
+            </geometry>
+            <material name="Cyan">
+                <color rgba="0 1.0 1.0 1.0"/>
+            </material>
+        </visual>
+        <collision>
+            <origin xyz="0 0 0" rpy="0 0 0"/>
+            <geometry>
+                <box size="0.05 0.1 0.1"/>
+            </geometry>
+        </collision>
+    </link>
+    <joint name="radar_joint" type="fixed">
+        <parent link="base_link"/>
+        <child link="/radar_link"/>
+        <origin xyz=" ${-0.48 - husky_rear_bumper_extend} 0 0.091" rpy="0 0 0" />
+    </joint>
     <!-- Husky wheel macros -->
     <xacro:husky_wheel wheel_prefix="${prefix}front_left">
@@ -147,5 +169,5 @@
           <param name="max_speed">1.0</param>
           <param name="polling_timeout">10.0</param>
-          <param name="serial_port">/dev/prolific</param>
+          <param name="serial_port">/dev/ttyUSB0</param>
         </xacro:unless>
       </hardware>
